Commit message: Began GUI testing

File: robonova/robot.urdf (robot description, URDF)
Before this commit: robot onshape, 13 links, 12 joints
Links:
- removed link base
- removed link cintura_urdf
- removed link cintura_urdf_2
- removed link femur_v01
- removed link femur_v01_2
- removed link pie_urdf
- removed link pie_urdf_2
- removed link tobillo_urdf
- removed link tobillo_urdf_2
- added link brazourdf, mass 1.080760232398511711; collision mesh filename=package:///brazo.stl; collision mesh filename=package:///motorejeacoplecaja.stl
- added link brazourdf_2, mass 1.080760232398511711; collision mesh filename=package:///brazo.stl; collision mesh filename=package:///motorejeacoplecaja.stl
- added link cintura_v01, mass 0.032703197933895256089; collision mesh filename=package:///cinturapt1.stl; collision mesh filename=package:///cinturapt2_1.stl
- added link cintura_v01_2, mass 0.032703197933895256089; collision mesh filename=package:///cinturapt1.stl; collision mesh filename=package:///cinturapt2_1.stl
- added link femururdf, mass 0.53868761965446410045; collision mesh filename=package:///femur.stl; collision mesh filename=package:///femur.stl
- added link femururdf_2, mass 0.53868761965446410045; collision mesh filename=package:///femur.stl; collision mesh filename=package:///femur.stl
- added link hombro-brazo, mass 0.028276359613946904642; collision mesh filename=package:///hombro_brazo1.stl; collision mesh filename=package:///hombro_brazo2.stl
- added link hombro-brazo_2, mass 0.028276359613946904642; collision mesh filename=package:///hombro_brazo1.stl; collision mesh filename=package:///hombro_brazo2.stl
- added link pieurdf, mass 0.12193030814742022994; collision mesh filename=package:///acoplepiemotor.stl; collision mesh filename=package:///acoplepiemotor.stl
- added link pieurdf_2, mass 0.12193030814742022994; collision mesh filename=package:///acoplepiemotor.stl; collision mesh filename=package:///acoplepiemotor.stl
- added link tobillourdf, mass 0.35953278469495458802; collision mesh filename=package:///motorejecaja.stl; collision mesh filename=package:///motorejeeje1.stl
- added link tobillourdf_2, mass 0.35953278469495464353; collision mesh filename=package:///motorejecaja.stl; collision mesh filename=package:///motorejeeje1.stl
- added link torsourdf, mass 3.2921674694110931725; collision mesh filename=package:///abdomen.stl; collision mesh filename=package:///acople_tornillos_abdomen.stl
- link cadera_v01: geometry collision mesh filename=package:///caderapt1.stl; collision mesh filename=package:///caderapt2_1.stl
- link cadera_v01_2: mass 0.36033150614011227875 -> 0.36033150614011233426; geometry collision mesh filename=package:///caderapt1.stl; collision mesh filename=package:///caderapt2_1.stl
- link tibiaurdf: geometry collision mesh filename=package:///motorejeacoplecaja.stl; collision mesh filename=package:///motorejeacopleeje1.stl
- link tibiaurdf_2: geometry collision mesh filename=package:///motorejeacoplecaja.stl; collision mesh filename=package:///motorejeacopleeje1.stl
Joints:
- added joint LeftShoulder1: type revolute, parent torsourdf, child hombro-brazo, origin xyz=0.092805821023547840909 0.0073712188771943082041 0.02546852102891152686 rpy=-1.5707963267948943376 -5.5511151231257851673e-17 1.570796326794896336, axis 0 0 1, limit lower=-1.570796326794896558 upper=1.570796326794896558 effort=1 velocity=20
- added joint LeftShoulder2: type revolute, parent hombro-brazo, child brazourdf, origin xyz=-0.023549999999996178157 3.805458519655358085e-07 -0.020946406845601492352 rpy=7.6131020406662958056e-15 -1.5707963267948694686 0, axis 0 0 1, limit lower=-0.26179938779914940783 upper=3.141592653589793116 effort=1 velocity=20
- added joint RightShoulder1: type revolute, parent torsourdf, child hombro-brazo_2, origin xyz=-0.085191785003578379687 0.0073712188771942830506 0.025468521028911540738 rpy=1.5707963267948954478 -1.6653345369376078533e-16 -1.5707963267948976682, axis 0 0 1, limit lower=-1.570796326794896558 upper=1.570796326794896558 effort=1 velocity=20
- added joint RightShoulder2: type revolute, parent hombro-brazo_2, child brazourdf_2, origin xyz=-0.023549999999995938765 -3.8054585671173923878e-07 0.018946406845602059565 rpy=3.1415926535894782567 1.5707963267948730213 0, axis 0 0 1, limit lower=-0.26179938779914940783 upper=3.141592653589793116 effort=1 velocity=20
- joint LeftAnkle1: child tobillo_urdf_2 -> tobillourdf; origin xyz=5.9674487573602164048e-16 -0.055000000000000437428 1.0408340855860842566e-17 rpy=-1.9609509983142411855e-15 1.8008263821212345284e-16 -3.1415926535897926719 -> xyz=2.7755575615628913511e-17 0.054999999999999882316 0.046799999999999897238 rpy=3.1415926535897868987 -2.4196156553935806658e-14 -3.1415926535897114036; parent tibiaurdf_2 -> tibiaurdf
- joint LeftAnkle2: child pie_urdf_2 -> pieurdf; origin xyz=-0.023200000000000386979 0.025773004946420954159 0.033535984972317398056 rpy=1.5707963267947531172 -1.3089969389957789581 1.5707963267949207609 -> xyz=0.023599999999999961287 0.025772450770437771439 0.033535984972323150399 rpy=2.037085777839408061e-14 -1.5707963267947913089 0; parent tobillo_urdf_2 -> tobillourdf
- joint LeftHip1: child cadera_v01_2 -> cadera_v01; limit lower=-0.34906585039886589561 upper=0.34906585039886589561 effort=1 velocity=20 -> lower=-0.52359877559829881566 upper=0.52359877559829881566 effort=1 velocity=20; origin xyz=0.0231499999999999935 0.022673904349987915319 -0.023580436102933310938 rpy=-1.178442120830790527e-15 1.5707963267948934494 0 -> xyz=0.02354999999999998414 0.022673904349987897971 -0.02360543610293333594 rpy=-2.1049685500540671756e-15 1.5707963267948954478 0; parent cintura_urdf_2 -> cintura_v01
- joint LeftHip2: child femur_v01_2 -> femururdf; origin xyz=0.028027549229578674339 0.033035984972317182506 -0.023550000000022431462 rpy=-1.570796326820399047 1.5370119106032991141 -2.574471375494626401e-11 -> xyz=0.028027549229560577704 -0.014064015027681592285 -0.023549999999998755956 rpy=1.5707963267948557018 1.5707963267948159558 0; parent cadera_v01_2 -> cadera_v01
- joint LeftKnee: child tibiaurdf_2 -> tibiaurdf; limit lower=-2.0943951023931952626 upper=0 effort=1 velocity=20 -> lower=-0.26179938779914940783 upper=2.356194490192344837 effort=1 velocity=20; origin xyz=-2.6541269182445148545e-15 -0.065000000000000612843 -1.360023205165816762e-15 rpy=-3.1415926535897917837 -2.1125392990547635288e-15 3.1415926535897638061 -> xyz=2.7755575615628913511e-17 0.065000000000000029976 2.0816681711721685133e-17 rpy=3.1415926535897926719 -1.1730918729772736225e-15 -3.1415926535897114036; parent femur_v01_2 -> femururdf
- joint LeftWaist: child cintura_urdf_2 -> cintura_v01; limit lower=-1.570796326794896558 upper=0.785398163397448279 effort=1 velocity=20 -> lower=-0.26179938779914940783 upper=0.26179938779914940783 effort=1 velocity=20; origin xyz=-0.067534747132801886682 0.022753615593456101573 0.17243857811634974442 rpy=-0.040591453589791937073 -7.9363599025938875266e-17 -1.57079632679489678 -> xyz=0.019257018009984725598 0.0083712188771943082249 -0.083178910040700965167 rpy=1.72907851597959344e-39 7.0653760931075006984e-40 -1.570796326794896558; parent base -> torsourdf
- joint RightAnkle1: child tobillo_urdf -> tobillourdf_2; limit lower=-0.52359877559829881566 upper=0.785398163397448279 effort=1 velocity=20 -> lower=-0.785398163397448279 upper=0.52359877559829881566 effort=1 velocity=20; origin xyz=9.0205620750793968909e-17 -0.054999999999999903133 5.5511151231257827021e-17 rpy=2.2549919000224758686e-15 1.6152720456270272169e-15 -3.1415926535897829019 -> xyz=8.6736173798840354721e-18 0.05500000000000004885 0.046799999999999994382 rpy=3.141592653589793116 4.3896650401099704644e-16 9.5660208773739903412e-16; parent tibiaurdf -> tibiaurdf_2
- joint RightAnkle2: child pie_urdf -> pieurdf_2; origin xyz=-0.023200000000000386979 0.025773004946420954159 0.033535984972317384178 rpy=-1.5707963267944831109 -1.4808651911478258878 -1.570796326795454112 -> xyz=-0.023199999999999894318 -0.02577245077043927024 0.013564015027679135472 rpy=-9.2675866980585320865e-14 1.5707963267947497865 0; parent tobillo_urdf -> tobillourdf_2
- joint RightHip1: child cadera_v01 -> cadera_v01_2; limit lower=-0.34906585039886589561 upper=0.34906585039886589561 effort=1 velocity=20 -> lower=-0.52359877559829881566 upper=0.52359877559829881566 effort=1 velocity=20; origin xyz=0.023150000000000128808 0.022673904349987922258 -0.023580436102933310938 rpy=-1.7849231868056687303e-15 1.5707963267948952257 0 -> xyz=-0.023550000000000039652 0.022673904349987825113 -0.02360543610293333594 rpy=3.1415926535897913396 1.5707963267948956698 0; parent cintura_urdf -> cintura_v01_2
- joint RightHip2: child femur_v01 -> femururdf_2; origin xyz=0.028027549229578702095 0.033035984972317189445 -0.023550000000022434932 rpy=-1.5707963268204001572 1.5370119106033031109 -2.5738881126654993852e-11 -> xyz=0.028027549229562395694 -0.033035984972319951125 -0.023250000000002636613 rpy=1.5707963267949076602 -1.5707963267948039654 0; parent cadera_v01 -> cadera_v01_2
- joint RightKnee: child tibiaurdf -> tibiaurdf_2; limit lower=0 upper=2.0943951023931952626 effort=1 velocity=20 -> lower=-0.26179938779914940783 upper=2.356194490192344837 effort=1 velocity=20; origin xyz=-2.4841240175987877592e-15 -0.065000000000000557332 -1.360023205165816762e-15 rpy=-3.1415926535897886751 -3.2856652020904885758e-15 3.1415864293030528742 -> xyz=-6.3664351568348820365e-16 -0.065000000000000168754 -1.3877787807814456755e-17 rpy=3.141592653589793116 6.0472093121809969072e-15 2.2482016248737809052e-15; parent femur_v01 -> femururdf_2
- joint RightWaist: child cintura_urdf -> cintura_v01_2; limit lower=-0.785398163397448279 upper=1.570796326794896558 effort=1 velocity=20 -> lower=-0.26179938779914940783 upper=0.26179938779914940783 effort=1 velocity=20; origin xyz=-0.097510035534551134373 0.022753615593456243821 0.1736559873457808878 rpy=0.040591453589792783618 -1.1502857612098471035e-16 1.5707963267948961139 -> xyz=-0.010742981990015255944 0.0083712188771943168986 -0.083178910040700979045 rpy=-1.2602862693222394471e-29 5.03337832939847449e-16 1.57079632679489678; parent base -> torsourdf
