Commit message: Updated URDF

File: Programacion/FinalVersion/robonova/robot.urdf (robot description, URDF)
Before this commit: robot onshape, 17 links, 16 joints
Links:
- link cadera_v01: mass 0.36033150614011227875 -> 0.36033150614011222324
- link cadera_v01_2: mass 0.36033150614011233426 -> 0.36033150614011227875
- link hombro-brazo: mass 0.028276359613946904642 -> 0.028276359613946901173
- link hombro-brazo_2: mass 0.028276359613946904642 -> 0.028276359613946901173
- link pieurdf: mass 0.12193030814742022994 -> 0.12193030814742024381
- link pieurdf_2: mass 0.12193030814742022994 -> 0.12193030814742024381
- link tibiaurdf_2: mass 0.28552673687099017208 -> 0.28552673687099011657
- link tobillourdf: mass 0.35953278469495458802 -> 0.35953278469495453251
- link tobillourdf_2: mass 0.35953278469495464353 -> 0.35953278469495453251
- link torsourdf: mass 3.2921674694110931725 -> 3.2921674694109959169
Joints:
- joint LeftAnkle1: limit lower=-0.785398163397448279 upper=0.52359877559829881566 effort=1 velocity=20 -> lower=-0.785398163397448279 upper=0.785398163397448279 effort=1 velocity=20; origin xyz=2.7755575615628913511e-17 0.054999999999999882316 0.046799999999999897238 rpy=3.1415926535897868987 -2.4196156553935806658e-14 -3.1415926535897114036 -> xyz=-0.047631397208144216071 0.027499999999999982792 0.046800000000000036016 rpy=3.141592653589793116 -3.3493042203660128646e-16 -2.0943951023931943745
- joint LeftAnkle2: origin xyz=0.023599999999999961287 0.025772450770437771439 0.033535984972323150399 rpy=2.037085777839408061e-14 -1.5707963267947913089 0 -> xyz=0.023600000000001168654 0.02577245077044121313 0.033535984972323733266 rpy=-1.5707963267949103248 -1.458647397724844641 1.5707963267951052799
- joint LeftHip1: limit lower=-0.52359877559829881566 upper=0.52359877559829881566 effort=1 velocity=20 -> lower=-0.785398163397448279 upper=0.785398163397448279 effort=1 velocity=20; origin xyz=0.02354999999999998414 0.022673904349987897971 -0.02360543610293333594 rpy=-2.1049685500540671756e-15 1.5707963267948954478 0 -> xyz=0.0006194931750873496068 0.032685236218794766483 -0.023605436102933349818 rpy=-0.7853981633975747334 1.5707963267948947816 0
- joint LeftHip2: origin xyz=0.028027549229560577704 -0.014064015027681592285 -0.023549999999998755956 rpy=1.5707963267948557018 1.5707963267948159558 0 -> xyz=0.02802754922956399164 -0.014064015027681252279 -0.023550000000000497619 rpy=1.5707963268454843142 1.5683459094928371425 5.0356913078067518828e-11
- joint LeftKnee: limit lower=-0.26179938779914940783 upper=2.356194490192344837 effort=1 velocity=20 -> lower=-1.0471975511965976313 upper=1.0471975511965976313 effort=1 velocity=20; origin xyz=2.7755575615628913511e-17 0.065000000000000029976 2.0816681711721685133e-17 rpy=3.1415926535897926719 -1.1730918729772736225e-15 -3.1415926535897114036 -> xyz=8.1532003370909933437e-17 0.064999999999999891198 1.561251128379126385e-16 rpy=3.1415926535897922278 -7.3910170491445287467e-16 -2.0943951023931952626
- joint LeftShoulder2: limit lower=-0.26179938779914940783 upper=3.141592653589793116 effort=1 velocity=20 -> lower=-1.570796326794896558 upper=1.570796326794896558 effort=1 velocity=20; origin xyz=-0.023549999999996178157 3.805458519655358085e-07 -0.020946406845601492352 rpy=7.6131020406662958056e-15 -1.5707963267948694686 0 -> xyz=-0.02354999999999616081 3.8054585194818857374e-07 -0.020946406845601450719 rpy=7.7715611723741378302e-15 -1.5707963267948685804 0
- joint LeftWaist: limit lower=-0.26179938779914940783 upper=0.26179938779914940783 effort=1 velocity=20 -> lower=-1.570796326794896558 upper=1.570796326794896558 effort=1 velocity=20; origin xyz=0.019257018009984725598 0.0083712188771943082249 -0.083178910040700965167 rpy=1.72907851597959344e-39 7.0653760931075006984e-40 -1.570796326794896558 -> xyz=0.019257018009984729068 0.0083712188771943168986 -0.083178910040700979045 rpy=1.2791997842974976649e-19 8.2453707267879112331e-20 -2.3781265927246031389
- joint RightAnkle1: origin xyz=8.6736173798840354721e-18 0.05500000000000004885 0.046799999999999994382 rpy=3.141592653589793116 4.3896650401099704644e-16 9.5660208773739903412e-16 -> xyz=-0.047631397208144327093 0.027500000000000093814 0.046800000000000861744 rpy=3.1415926535897922278 -5.3373354253318456839e-16 1.832595714594138725
- joint RightAnkle2: origin xyz=-0.023199999999999894318 -0.02577245077043927024 0.013564015027679135472 rpy=-9.2675866980585320865e-14 1.5707963267947497865 0 -> xyz=-0.023200000000000303713 -0.025772450770438881662 0.013564015027679159758 rpy=-1.5707963267949147657 1.5122843990177565754 -1.5707963267948334973
- joint RightHip1: limit lower=-0.52359877559829881566 upper=0.52359877559829881566 effort=1 velocity=20 -> lower=-0.785398163397448279 upper=0.785398163397448279 effort=1 velocity=20; origin xyz=-0.023550000000000039652 0.022673904349987825113 -0.02360543610293333594 rpy=3.1415926535897913396 1.5707963267948956698 0 -> xyz=-0.00061949317509168121132 0.032685236218795189755 -0.023605436102933877174 rpy=-2.3561944901923315143 1.5707963267948703567 0
- joint RightHip2: origin xyz=0.028027549229562395694 -0.033035984972319951125 -0.023250000000002636613 rpy=1.5707963267949076602 -1.5707963267948039654 0 -> xyz=0.028027549229562506716 -0.033035984972318972741 -0.023249999999999167166 rpy=1.5707963267949034414 -1.5707963267948585884 0
- joint RightKnee: limit lower=-0.26179938779914940783 upper=2.356194490192344837 effort=1 velocity=20 -> lower=-1.0471975511965976313 upper=1.0471975511965976313 effort=1 velocity=20; origin xyz=-6.3664351568348820365e-16 -0.065000000000000168754 -1.3877787807814456755e-17 rpy=3.141592653589793116 6.0472093121809969072e-15 2.2482016248737809052e-15 -> xyz=2.8449465006019636348e-16 -0.065000000000000363043 -1.0824674490095276269e-15 rpy=3.1415926535897717997 9.8745822879544016264e-15 1.0471975511965985195
- joint RightShoulder1: origin xyz=-0.085191785003578379687 0.0073712188771942830506 0.025468521028911540738 rpy=1.5707963267948954478 -1.6653345369376078533e-16 -1.5707963267948976682 -> xyz=-0.085191785003578324176 0.0073712188771942856527 0.025468521028911415838 rpy=1.57079632679489678 -2.222614453594627363e-16 -1.57079632679489678
- joint RightShoulder2: limit lower=-0.26179938779914940783 upper=3.141592653589793116 effort=1 velocity=20 -> lower=-1.570796326794896558 upper=1.570796326794896558 effort=1 velocity=20; origin xyz=-0.023549999999995938765 -3.8054585671173923878e-07 0.018946406845602059565 rpy=3.1415926535894782567 1.5707963267948730213 0 -> xyz=-0.023549999999995352429 -3.8054585540028829094e-07 0.018946406845602128954 rpy=3.1415926535894787008 1.5707963267948730213 0
- joint RightWaist: limit lower=-0.26179938779914940783 upper=0.26179938779914940783 effort=1 velocity=20 -> lower=-1.570796326794896558 upper=1.570796326794896558 effort=1 velocity=20; origin xyz=-0.010742981990015255944 0.0083712188771943168986 -0.083178910040700979045 rpy=-1.2602862693222394471e-29 5.03337832939847449e-16 1.57079632679489678 -> xyz=-0.010742981990015255944 0.0083712188771943168986 -0.083178910040700979045 rpy=5.0065502374750631335e-32 4.1312151660743903538e-31 2.3608809754637762879

Commit message: Updated URDF

File: Programacion/FinalVersion/robonova/robot.urdf (robot description, URDF)
Before this commit: robot onshape, 17 links, 16 joints
Links:
- link pieurdf: mass 0.12193030814742024381 -> 0.12193030814742020218
- link pieurdf_2: mass 0.12193030814742024381 -> 0.12193030814742020218
- link tobillourdf: mass 0.35953278469495453251 -> 0.35953278469495458802
- link torsourdf: mass 3.2921674694109959169 -> 3.292167469410996361
Joints:
- joint LeftAnkle1: origin xyz=-0.047631397208144216071 0.027499999999999982792 0.046800000000000036016 rpy=3.141592653589793116 -3.3493042203660128646e-16 -2.0943951023931943745 -> xyz=-0.047631397208144299338 0.027499999999999968914 0.04680000000000013316 rpy=3.1415926535897922278 -8.3236563318828217705e-16 -2.0943951023931934863
- joint LeftAnkle2: origin xyz=0.023600000000001168654 0.02577245077044121313 0.033535984972323733266 rpy=-1.5707963267949103248 -1.458647397724844641 1.5707963267951052799 -> xyz=0.023600000000001175593 0.025772450770441185375 0.033535984972323726327 rpy=1.9660785197239803745e-13 -1.5707963267947935293 0
- joint LeftKnee: origin xyz=8.1532003370909933437e-17 0.064999999999999891198 1.561251128379126385e-16 rpy=3.1415926535897922278 -7.3910170491445287467e-16 -2.0943951023931952626 -> xyz=-1.2143064331837649661e-16 0.064999999999999863443 1.7694179454963432363e-16 rpy=-3.141592653589793116 -1.2372584350642698768e-15 -3.1415926535897922278
- joint RightAnkle1: origin xyz=-0.047631397208144327093 0.027500000000000093814 0.046800000000000861744 rpy=3.1415926535897922278 -5.3373354253318456839e-16 1.832595714594138725 -> xyz=-0.047631397208144188316 0.027500000000000524025 0.046800000000001645839 rpy=3.1415926535897913396 -1.289442150517726367e-15 1.0471975511965989636
- joint RightAnkle2: origin xyz=-0.023200000000000303713 -0.025772450770438881662 0.013564015027679159758 rpy=-1.5707963267949147657 1.5122843990177565754 -1.5707963267948334973 -> xyz=-0.023200000000000164935 -0.025772450770439048195 0.013564015027679472009 rpy=-9.2634305154051540682e-14 1.570796326794752007 0
- joint RightKnee: origin xyz=2.8449465006019636348e-16 -0.065000000000000363043 -1.0824674490095276269e-15 rpy=3.1415926535897717997 9.8745822879544016264e-15 1.0471975511965985195 -> xyz=2.3765711620882257193e-16 -0.065000000000000474065 -9.7144514654701197287e-16 rpy=-3.1415926535897855665 6.6257119499898968432e-15 4.6469541351745896613e-16

Commit message: Buttons that recieve and send data complete.

File: Programacion/FinalVersion/robonova/robot.urdf (robot description, URDF)
Before this commit: robot onshape, 17 links, 16 joints
Links:
- link pieurdf: mass 0.12193030814742020218 -> 0.12193030814742022994
- link pieurdf_2: mass 0.12193030814742020218 -> 0.12193030814742022994
- link torsourdf: mass 3.292167469410996361 -> 3.2921674694110931725
Joints:
- joint LeftAnkle1: origin xyz=-0.047631397208144299338 0.027499999999999968914 0.04680000000000013316 rpy=3.1415926535897922278 -8.3236563318828217705e-16 -2.0943951023931934863 -> xyz=-0.047631397208144125865 0.027499999999999968914 0.046800000000000036016 rpy=-3.1415926535897917837 -4.9721604402088067868e-16 -2.0943951023931961508
- joint LeftAnkle2: origin xyz=0.023600000000001175593 0.025772450770441185375 0.033535984972323726327 rpy=1.9660785197239803745e-13 -1.5707963267947935293 0 -> xyz=0.023600000000001231104 0.025772450770440658019 0.033535984972325266762 rpy=1.5454106253939043597e-13 -1.5707963267947788744 0
- joint LeftHip1: origin xyz=0.0006194931750873496068 0.032685236218794766483 -0.023605436102933349818 rpy=-0.7853981633975747334 1.5707963267948947816 0 -> xyz=0.0006194931750914097271 0.03268523621879472485 -0.023605436102933363696 rpy=-0.78539816339744661366 1.5707963267948883423 0
- joint LeftHip2: origin xyz=0.02802754922956399164 -0.014064015027681252279 -0.023550000000000497619 rpy=1.5707963268454843142 1.5683459094928371425 5.0356913078067518828e-11 -> xyz=0.028027549229563922251 -0.014064015027682230663 -0.023550000000002006828 rpy=1.570796326794806852 1.5707963267946500885 0
- joint LeftKnee: origin xyz=-1.2143064331837649661e-16 0.064999999999999863443 1.7694179454963432363e-16 rpy=-3.141592653589793116 -1.2372584350642698768e-15 -3.1415926535897922278 -> xyz=-5.898059818321144121e-17 0.065000000000000196509 -7.147060721024445229e-16 rpy=-3.1415926535897926719 9.8471969112908084787e-16 -3.1415926535897922278
- joint LeftWaist: origin xyz=0.019257018009984729068 0.0083712188771943168986 -0.083178910040700979045 rpy=1.2791997842974976649e-19 8.2453707267879112331e-20 -2.3781265927246031389 -> xyz=0.019257018009984729068 0.0083712188771943168986 -0.083178910040700979045 rpy=-4.9415502631049690248e-17 6.1232339957363309298e-17 -1.570796326794896558
- joint RightAnkle1: origin xyz=-0.047631397208144188316 0.027500000000000524025 0.046800000000001645839 rpy=3.1415926535897913396 -1.289442150517726367e-15 1.0471975511965989636 -> xyz=-0.047631397208144354849 0.027499999999999885647 0.046800000000000029077 rpy=-3.1415926535897908956 -2.4069865602134688359e-15 1.0471975511965929684
- joint RightAnkle2: origin xyz=-0.023200000000000164935 -0.025772450770439048195 0.013564015027679472009 rpy=-9.2634305154051540682e-14 1.570796326794752007 0 -> xyz=-0.023200000000000831069 -0.025772450770438881662 0.013564015027679409559 rpy=-9.8713777730327891289e-14 1.5707963267947468999 0
- joint RightHip1: origin xyz=-0.00061949317509168121132 0.032685236218795189755 -0.023605436102933877174 rpy=-2.3561944901923315143 1.5707963267948703567 0 -> xyz=-0.00061949317509201601295 0.032685236218795134244 -0.023605436102933322062 rpy=-2.3561944901923403961 1.570796326794891673 0
- joint RightHip2: origin xyz=0.028027549229562506716 -0.033035984972318972741 -0.023249999999999167166 rpy=1.5707963267949034414 -1.5707963267948585884 0 -> xyz=0.028027549229562492838 -0.03303598497231897968 -0.023249999999999160227 rpy=1.5707963267949229813 -1.5707963267948594765 0
- joint RightKnee: origin xyz=2.3765711620882257193e-16 -0.065000000000000474065 -9.7144514654701197287e-16 rpy=-3.1415926535897855665 6.6257119499898968432e-15 4.6469541351745896613e-16 -> xyz=1.3053794156725473385e-16 -0.064999999999999807931 -1.0963452368173420837e-15 rpy=3.1415926535897895633 -5.1908057209288357076e-17 3.6528103707004495366e-15
- joint RightWaist: origin xyz=-0.010742981990015255944 0.0083712188771943168986 -0.083178910040700979045 rpy=5.0065502374750631335e-32 4.1312151660743903538e-31 2.3608809754637762879 -> xyz=-0.010742981990015255944 0.0083712188771943186333 -0.083178910040700965167 rpy=5.1336160526084935663e-31 -6.2213430271953116103e-32 1.5707963267948970021

Commit message: URDF changed, dials for loop done

File: Programacion/FinalVersion/robonova/robot.urdf (robot description, URDF)
Before this commit: robot onshape, 17 links, 16 joints
Links:
- link cadera_v01: mass 0.36033150614011222324 -> 0.36033150614011227875
- link cadera_v01_2: mass 0.36033150614011227875 -> 0.36033150614011233426
- link pieurdf: mass 0.12193030814742022994 -> 0.12193030814742021606
- link pieurdf_2: mass 0.12193030814742022994 -> 0.12193030814742021606
- link tibiaurdf_2: mass 0.28552673687099011657 -> 0.28552673687099017208
- link tobillourdf: mass 0.35953278469495458802 -> 0.35953278469495453251
- link torsourdf: mass 3.2921674694110931725 -> 3.2921674694110936166
Joints:
- joint LeftAnkle1: origin xyz=-0.047631397208144125865 0.027499999999999968914 0.046800000000000036016 rpy=-3.1415926535897917837 -4.9721604402088067868e-16 -2.0943951023931961508 -> xyz=-0.04763139720814472261 0.027500000000000357492 0.046799999999997926592 rpy=3.141592653589793116 5.3675190344367677838e-16 -2.0943951023932081412
- joint LeftAnkle2: origin xyz=0.023600000000001231104 0.025772450770440658019 0.033535984972325266762 rpy=1.5454106253939043597e-13 -1.5707963267947788744 0 -> xyz=0.023600000000001397638 0.02577245077045106636 0.033535984972326855769 rpy=2.2132700711385145215e-13 -1.570796326794244635 0
- joint LeftHip1: origin xyz=0.0006194931750914097271 0.03268523621879472485 -0.023605436102933363696 rpy=-0.78539816339744661366 1.5707963267948883423 0 -> xyz=0.00061949317509150773897 0.032685236218795377106 -0.023605436102933363696 rpy=-0.78539816339745072149 1.5707963267948956698 0
- joint LeftHip2: origin xyz=0.028027549229563922251 -0.014064015027682230663 -0.023550000000002006828 rpy=1.570796326794806852 1.5707963267946500885 0 -> xyz=0.028027549229571513401 -0.014064015027672766012 -0.023549999999991647059 rpy=1.5707963267946409847 1.5707963267945965757 0
- joint LeftKnee: origin xyz=-5.898059818321144121e-17 0.065000000000000196509 -7.147060721024445229e-16 rpy=-3.1415926535897926719 9.8471969112908084787e-16 -3.1415926535897922278 -> xyz=-2.1510571102112407971e-16 0.065000000000001029177 -7.5980888247784150735e-16 rpy=-3.1415926535897904515 -9.7897424329627288022e-15 3.1415926535897908956
- joint LeftWaist: origin xyz=0.019257018009984729068 0.0083712188771943168986 -0.083178910040700979045 rpy=-4.9415502631049690248e-17 6.1232339957363309298e-17 -1.570796326794896558 -> xyz=0.019257018009984791518 0.0083712188771943828181 -0.083178910040700979045 rpy=-7.0498275397804529719e-24 -1.2781389790328887556e-24 -1.570796326794896558
- joint RightAnkle1: limit lower=-0.785398163397448279 upper=0.52359877559829881566 effort=1 velocity=20 -> lower=-0.785398163397448279 upper=0.785398163397448279 effort=1 velocity=20; origin xyz=-0.047631397208144354849 0.027499999999999885647 0.046800000000000029077 rpy=-3.1415926535897908956 -2.4069865602134688359e-15 1.0471975511965929684 -> xyz=-0.047631397208144729549 0.027500000000000440759 0.046799999999998891098 rpy=-3.141592653589793116 -8.7370753692816634214e-18 1.0471975511965838646
- joint RightAnkle2: origin xyz=-0.023200000000000831069 -0.025772450770438881662 0.013564015027679409559 rpy=-9.8713777730327891289e-14 1.5707963267947468999 0 -> xyz=-0.023200000000000914335 -0.025772450770440075152 0.013564015027678882203 rpy=-1.1383176501975356648e-13 1.5707963267947862018 0
- joint RightHip1: origin xyz=-0.00061949317509201601295 0.032685236218795134244 -0.023605436102933322062 rpy=-2.3561944901923403961 1.570796326794891673 0 -> xyz=-0.00061949317509176534541 0.032685236218794461172 -0.023605436102933266551 rpy=-2.3561944901923457252 1.5707963267948956698 0
- joint RightHip2: origin xyz=0.028027549229562492838 -0.03303598497231897968 -0.023249999999999160227 rpy=1.5707963267949229813 -1.5707963267948594765 0 -> xyz=0.028027549229563658573 -0.033035984972319389075 -0.023250000000002678247 rpy=1.5707963267949249797 -1.5707963267948361619 0
- joint RightKnee: origin xyz=1.3053794156725473385e-16 -0.064999999999999807931 -1.0963452368173420837e-15 rpy=3.1415926535897895633 -5.1908057209288357076e-17 3.6528103707004495366e-15 -> xyz=-2.0903417885520525488e-16 -0.065000000000000418554 -2.0816681711721685133e-16 rpy=3.1415926535897913396 -8.8716665251345430742e-16 -6.587726272486626974e-15
- joint RightWaist: origin xyz=-0.010742981990015255944 0.0083712188771943186333 -0.083178910040700965167 rpy=5.1336160526084935663e-31 -6.2213430271953116103e-32 1.5707963267948970021 -> xyz=-0.010742981990015255944 0.0083712188771943186333 -0.083178910040700992923 rpy=1.5914679956727636981e-17 5.1509014745192104691e-18 1.5707963267948981123
